File: Rp2350Board.kicad_sch (KiCad schematic)
At the start: 42 parts, among them J1 Conn_01x04, J2 Conn_01x02, J3 Conn_01x02, J4 Conn_01x06, J5 Conn_01x06, SW1 SW_Push, SW2 SW_Push, U1 RP2350A-QFN60, U2 LD1117V33, U3 W25Q128JVS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

Commit message: First draft of v2 board
Parts:
- removed C4: 100n, Capacitor_SMD:C_0603_1608Metric, symbol Device:C
- removed C5: 10u, Capacitor_SMD:C_0603_1608Metric, symbol Device:C
- removed J1: Conn_01x04, Connector_JST:JST_PH_B4B-PH-K_1x04_P2.00mm_Vertical, symbol Connector_Generic:Conn_01x04
- removed J4, J5: Conn_01x06, Connector_JST:JST_PH_B6B-PH-K_1x06_P2.00mm_Vertical, symbol Connector_Generic:Conn_01x06
- removed SW1, SW2: SW_Push, ProjectLibrary:SW_TL1015AF160QG, symbol Switch:SW_Push
- removed U2: LD1117V33, Package_TO_SOT_THT:TO-220-3_Vertical, symbol Regulator_Linear:LD1117V33
- added C21: 10u, Capacitor_SMD:C_0603_1608Metric, symbol Device:C
- added C22, C23: 22u, Capacitor_SMD:C_0603_1608Metric, symbol Device:C
- added C24: 100n, Capacitor_SMD:C_0603_1608Metric, symbol Device:C
- added J1, J6: Conn_01x02, Connector_JST:JST_GH_SM02B-GHS-TB_1x02-1MP_P1.25mm_Horizontal, symbol Connector_Generic:Conn_01x02
- added J4: Conn_01x10, Connector_PinSocket_2.00mm:PinSocket_1x10_P2.00mm_Vertical_SMD_Pin1Left, symbol Connector_Generic:Conn_01x10
- added J5: Conn_01x04, Connector_PinSocket_2.00mm:PinSocket_1x04_P2.00mm_Vertical_SMD_Pin1Left, symbol Connector_Generic:Conn_01x04
- added L2: L, symbol Device:L
- added S1, S2: EVQ-P7A01P, ProjectLibrary:SW_EVQ-P7A01P, symbol EVQ-P7A01P:EVQ-P7A01P
- added U2: AP63203WU, Package_TO_SOT_SMD:TSOT-23-6, symbol Regulator_Switching:AP63203WU
- J2, J3: footprint Connector_JST:JST_PH_B2B-PH-K_1x02_P2.00mm_Vertical -> Connector_JST:JST_GH_SM02B-GHS-TB_1x02-1MP_P1.25mm_Horizontal
- Y1: footprint ABM8-272-T3:XTAL_ABM8-272-T3 -> ProjectLibrary:XTAL_ABM8-272-T3
Connections:
- net +3V3: now also C22.2, C23.1, J5.3 (Pin_3), L2.2, U2.1 (FB)
- net GND: now also C21.2, C22.1, C23.2, J1.2 (Pin_2), J5.1 (Pin_1), J5.4 (Pin_4), S1.1_1, S1.1_2, S2.1_1, S2.1_2, U2.4 (GND)
- net USB D+: now also J6.1 (Pin_1)
- net USB D-: now also J6.2 (Pin_2)
- net USB_BOOT: now also S1.2_1, S1.2_2
- net at U1.27 (GPIO16): now also J4.1 (Pin_1)
- net at U1.28 (GPIO17): now also J4.2 (Pin_2)
- net at U1.29 (GPIO18): now also J4.3 (Pin_3)
- net at U1.31 (GPIO19): now also J4.4 (Pin_4)
- net at U1.32 (GPIO20): now also J4.5 (Pin_5)
- net at U1.37 (GPIO25): now also J4.6 (Pin_6)
- net at U1.40 (GPIO26_ADC0): now also J4.7 (Pin_7)
- net at U1.41 (GPIO27_ADC1): now also J4.8 (Pin_8)
- net at U1.42 (GPIO28_ADC2): now also J4.9 (Pin_9)
- net at U1.43 (GPIO29_ADC3): now also J4.10 (Pin_10)
- net RST: now reaches R5.1
- net RST: now also S2.2_1, S2.2_2
- new net: C24.1, L2.1, U2.5 (SW)
- new net: C24.2, U2.6 (BST)
- new net VBUS: C21.1, J1.1 (Pin_1), J5.2 (Pin_2), U2.2 (EN), U2.3 (IN)

Commit message: Small edits to first draft of v2
Parts:
- L2: footprint (none) -> ProjectLibrary:PA5430
Connections:
- net REG_SW: now reaches C24.1, L2.1, U2.5 (SW)
Changed lines of the file:
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@@
 		)
 	)
+	(label "REG_SW"
+		(at 100.33 35.56 0)
+		(effects
+			(font
+				(size 1.27 1.27)
+			)
+			(justify left bottom)
+		)
+	)
 	(label "VREG"
 		(at 27.94 97.79 0)
@@
 			)
 		)
-		(property "Footprint" ""
+		(property "Footprint" "ProjectLibrary:PA5430"
 			(at 111.76 35.56 0)
 			(effects

Commit message: Small fixups and cleanup of unused external library files
Parts:
- removed S1, S2: EVQ-P7A01P, ProjectLibrary:SW_EVQ-P7A01P, symbol EVQ-P7A01P:EVQ-P7A01P
- added SW1, SW2: SW_Push, ProjectLibrary:SW_EVQ-P7A01P, symbol Switch:SW_Push
Connections:
- net GND: now also SW1.1_1 (1), SW2.1_1 (1)
- net RST: now also SW2.2_1 (2)
- net USB_BOOT: now also SW1.2_1 (2)
